Commit message: edo kin & dyn 6link

File: edo/implementation/simulator_edo/robots/edo_sim.urdf (robot description, URDF)
Before this commit: robot simulator_edo, 7 links, 6 joints
Joints:
- joint joint_4: type fixed -> continuous
- joint joint_5: type fixed -> continuous
- joint joint_6: type fixed -> continuous
